File: hardware/Self_Watering_POT/Self_Watering_POT.kicad_pcb (KiCad board)
At the start: 2 copper layers, 50 x 80 mm, 70 parts, among them J1 Barrel_Jack, J5 Screw_Terminal_01x02, J6 Screw_Terminal_01x02, M2 MountingHole, Q1 IRLZ540N, SW1 SW_Push, SW2 SW_Push, SW3 SW_Push, U1 AMS1117-3.3_SOT223, U2 STM32F446RETx

Commit message: Corrected mistakes with PCB board
Parts:
- moved D4 1.29 mm to (184.7, 49.7)
- turned C1 to 180 degrees
- turned D2 to 90 degrees
- turned F1 to 0 degrees
Connections:
- D2 pad 1: GND -> /VIN_FUSED
- D2 pad 2: +12V -> GND
- D3 pad 2: +12V -> /VIN_FUSED
- D4 pad 2: +12V -> /PUMP_NEG
- F1 pad 1: +12V -> /VIN_RAW
- F1 pad 2: +12V -> /VIN_FUSED
- J1 pad 1: +12V -> /VIN_RAW
- J6 pad 1: +12V -> /PUMP_NEG
- Q1 pad 2: +12V -> /PUMP_NEG
Routing:
- net +12V: track 85.0 -> 35.0 mm
- net /PUMP_NEG: track 0.00 -> 25.0 mm
- net /VIN_RAW: track 0.00 -> 10.3 mm
- net /VIN_FUSED: track 0.00 -> 9.74 mm
