File: hardware/Self_Watering_POT/Self_Watering_POT.kicad_sch (KiCad schematic)
At the start: 69 parts, among them J1 Barrel_Jack, J5 Screw_Terminal_01x02, J6 Screw_Terminal_01x02, M2 MountingHole, Q1 IRLZ540N, SW1 SW_Push, SW2 SW_Push, SW3 SW_Push, U1 AMS1117-3.3_SOT223, U2 STM32F446RETx

Commit message: Corrected mistakes with PCB board
Parts:
- C1, C3: symbol Device:C_Small -> Device:C_Polarized
Connections:
- net +12V: no longer D2.2 (A2), D3.2 (A), D4.2 (A), F1.1, F1.2, J1.1, J6.1 (Pin_1), Q1.2 (D)
- net GND: now also D2.2 (A2); no longer D2.1 (A1)
- new net PUMP_NEG: D4.2 (A), J6.1 (Pin_1), Q1.2 (D)
- new net VIN_FUSED: D2.1 (A1), D3.2 (A), F1.2
- new net VIN_RAW: F1.1, J1.1
Other:
- moved on the sheet: D2
Changed lines of the file:
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@@
 	)
 	(junction
-		(at 123.19 36.83)
-		(diameter 0)
-		(color 0 0 0 0)
-	)
-	(junction
-		(at 158.75 36.83)
-		(diameter 0)
-		(color 0 0 0 0)
-	)
-	(junction
 		(at 257.81 100.33)
 		(diameter 0)
@@
 	)
 	(junction
-		(at 158.75 53.34)
-		(diameter 0)
-		(color 0 0 0 0)
-	)
-	(junction
 		(at 171.45 102.87)
 		(diameter 0)
@@
 	)
 	(junction
+		(at 123.19 53.34)
+		(diameter 0)
+		(color 0 0 0 0)
+	)
+	(junction
 		(at 95.25 210.82)
 		(diameter 0)
@@
 	)
 	(junction
+		(at 158.75 36.83)
+		(diameter 0)
+		(color 0 0 0 0)
+	)
+	(junction
 		(at 194.31 107.95)
 		(diameter 0)
@@
 	)
 	(junction
+		(at 158.75 53.34)
+		(diameter 0)
+		(color 0 0 0 0)
+	)
+	(junction
+		(at 123.19 36.83)
+		(diameter 0)
+		(color 0 0 0 0)
+	)
+	(junction
 		(at 182.88 102.87)
 		(diameter 0)
@@
 	)
 	(junction
-		(at 123.19 53.34)
-		(diameter 0)
-		(color 0 0 0 0)
-	)
-	(junction
 		(at 288.29 163.83)
 		(diameter 0)
@@
 	(wire
 		(pts
-			(xy 123.19 43.18) (xy 123.19 36.83)
-		)
-		(stroke
-			(width 0)
-			(type default)
-		)
-	)
-	(wire
-		(pts
 			(xy 90.17 99.06) (xy 90.17 114.3)
 		)
@@
 	(wire
 		(pts
-			(xy 158.75 36.83) (xy 177.8 36.83)
+			(xy 149.86 36.83) (xy 158.75 36.83)
 		)
 		(stroke
@@
 	(wire
 		(pts
-			(xy 123.19 48.26) (xy 123.19 53.34)
+			(xy 127 36.83) (xy 134.62 36.83)
 		)
 		(stroke
@@
 	(wire
 		(pts
-			(xy 127 36.83) (xy 134.62 36.83)
+			(xy 262.89 48.26) (xy 292.1 48.26)
 		)
 		(stroke
@@
 	(wire
 		(pts
-			(xy 262.89 48.26) (xy 292.1 48.26)
+			(xy 212.09 175.26) (xy 212.09 181.61)
 		)
 		(stroke
@@
 	(wire
 		(pts
-			(xy 212.09 175.26) (xy 212.09 181.61)
+			(xy 64.77 256.54) (xy 69.85 256.54)
 		)
 		(stroke
@@
 	(wire
 		(pts
-			(xy 64.77 256.54) (xy 69.85 256.54)
+			(xy 274.32 166.37) (xy 267.97 166.37)
 		)
 		(stroke
@@
 	(wire
 		(pts
-			(xy 274.32 166.37) (xy 267.97 166.37)
+			(xy 158.75 36.83) (xy 158.75 41.91)
 		)
 		(stroke
@@
 		)
 	)
-	(wire
-		(pts
-			(xy 158.75 48.26) (xy 158.75 53.34)
-		)
-		(stroke
-			(width 0)
-			(type default)
-		)
-	)
 	(polyline
 		(pts
@@
 	(wire
 		(pts
+			(xy 158.75 53.34) (xy 177.8 53.34)
+		)
+		(stroke
+			(width 0)
+			(type default)
+		)
+	)
+	(wire
+		(pts
 			(xy 177.8 53.34) (xy 186.69 53.34)
 		)
@@
 	(wire
 		(pts
-			(xy 149.86 36.83) (xy 158.75 36.83)
-		)
-		(stroke
-			(width 0)
-			(type default)
-		)
-	)
-	(wire
-		(pts
 			(xy 63.5 177.8) (xy 74.93 177.8)
 		)
@@
 	(wire
 		(pts
-			(xy 158.75 53.34) (xy 177.8 53.34)
-		)
-		(stroke
-			(width 0)
-			(type default)
-		)
-	)
-	(wire
-		(pts
 			(xy 95.25 210.82) (xy 95.25 214.63)
 		)
@@
 	(wire
 		(pts
+			(xy 123.19 36.83) (xy 123.19 41.91)
+		)
+		(stroke
+			(width 0)
+			(type default)
+		)
+	)
+	(wire
+		(pts
 			(xy 274.32 181.61) (xy 274.32 173.99)
 		)
@@
 	(wire
 		(pts
+			(xy 158.75 36.83) (xy 177.8 36.83)
+		)
+		(stroke
+			(width 0)
+			(type default)
+		)
+	)
+	(wire
+		(pts
 			(xy 262.89 193.04) (xy 262.89 186.69)
 		)
@@
 	(wire
 		(pts
+			(xy 158.75 49.53) (xy 158.75 53.34)
+		)
+		(stroke
+			(width 0)
+			(type default)
+		)
+	)
+	(wire
+		(pts
 			(xy 274.32 203.2) (xy 274.32 207.01)
 		)
@@
 	(wire
 		(pts
-			(xy 158.75 43.18) (xy 158.75 36.83)
+			(xy 379.73 228.6) (xy 379.73 231.14)
 		)
 		(stroke
@@
 	(wire
 		(pts
-			(xy 379.73 228.6) (xy 379.73 231.14)
+			(xy 123.19 49.53) (xy 123.19 53.34)
 		)
 		(stroke
@@
 	)
 	(label "+12V"
-		(at 39.37 40.64 0)
+		(at 88.9 40.64 0)
 		(effects
 			(font
@@
 		)
 	)
-	(label "+12V"
-		(at 62.23 40.64 0)
+	(label "VIN_RAW"
+		(at 38.1 40.64 0)
 		(effects
 			(font
@@
 		)
 	)
-	(label "+12V"
-		(at 278.13 173.99 0)
+	(label "VIN_FUSED"
+		(at 53.34 40.64 0)
+		(effects
+			(font
+				(size 1.27 1.27)
+			)
+			(justify left bottom)
+		)
+	)
+	(label "PUMP_NEG"
+		(at 275.59 173.99 0)
 		(effects
 			(font
@@
 	(symbol
 		(lib_id "Device:D_TVS")
-		(at 62.23 49.53 90)
+		(at 62.23 49.53 270)
 		(unit 1)
 		(body_style 1)
@@
 					(size 1.27 1.27)
 				)
-				(justify right)
+				(justify left)
 			)
 		)
@@
 					(size 1.27 1.27)
 				)
-				(justify right)
+				(justify left)
 			)
 		)
@@
 	)
 	(symbol
-		(lib_id "Device:C_Small")
+		(lib_id "Device:C_Polarized")
 		(at 158.75 45.72 0)
 		(unit 1)
@@
 		(fields_autoplaced yes)
 		(property "Reference" "C3"
-			(at 161.29 44.4562 0)
+			(at 162.56 43.5609 0)
 			(show_name no)
 			(do_not_autoplace no)
@@
 		)
 		(property "Value" "10uF"
-			(at 161.29 46.9962 0)
+			(at 162.56 46.1009 0)
 			(show_name no)
 			(do_not_autoplace no)
@@
 		)
 		(property "Footprint" "Capacitor_Tantalum_SMD:CP_EIA-3216-18_Kemet-A"
-			(at 158.75 45.72 0)
+			(at 159.7152 49.53 0)
 			(hide yes)
 			(show_name no)
@@
 			)
 		)
-		(property "Description" "Unpolarized capacitor, small symbol"
+		(property "Description" "Polarized capacitor"
 			(at 158.75 45.72 0)
 			(hide yes)
@@
 	)
 	(symbol
-		(lib_id "Device:C_Small")
+		(lib_id "Device:C_Polarized")
 		(at 123.19 45.72 0)
 		(unit 1)
@@
 		(fields_autoplaced yes)
 		(property "Reference" "C1"
-			(at 125.73 44.4562 0)
+			(at 127 43.5609 0)
 			(show_name no)
 			(do_not_autoplace no)
@@
 		)
 		(property "Value" "10uF"
-			(at 125.73 46.9962 0)
+			(at 127 46.1009 0)
 			(show_name no)
 			(do_not_autoplace no)
@@
 		)
 		(property "Footprint" "Capacitor_Tantalum_SMD:CP_EIA-3216-18_Kemet-A"
-			(at 123.19 45.72 0)
+			(at 124.1552 49.53 0)
 			(hide yes)
 			(show_name no)
@@
 			)
 		)
-		(property "Description" "Unpolarized capacitor, small symbol"
+		(property "Description" "Polarized capacitor"
 			(at 123.19 45.72 0)
 			(hide yes)
